Commit message: add: Lidar

File: urdf/microbot_01_base.xacro (robot description, xacro)
@@ -23,3 +23,30 @@
     </visual>
   </link>
+ <xacro:property name="laser_d" value="0.06" />
+  <xacro:property name="laser_w" value="0.06" />
+  <xacro:property name="laser_h" value="0.06" />
+  <xacro:property name="laser_x" value="-0.0475" />
+  <xacro:property name="laser_z" value="${body_h}" />
+  <joint name="laser_joint" type="fixed">
+    <origin xyz="${laser_x} 0 ${laser_z}" rpy="0 0 0"/>
+    <parent link="base_link"/>
+    <child link="base_laser_link"/>
+  </joint>
+  <link name="base_laser_link">
+    <collision>
+      <origin rpy="0 0 0" xyz="0 0 0"/>
+      <geometry>
+        <box size="${laser_d} ${laser_w} ${laser_h}"/>
+      </geometry>
+    </collision>
+    <visual>
+      <origin rpy="0 0 0" xyz="0 0 0"/>
+      <geometry>
+        <box size="${laser_d} ${laser_w} ${laser_h}"/>
+      </geometry>
+      <material name="laser_mat">
+        <color rgba="0.0 0.0 0.0 0.8"/>
+      </material>
+    </visual>
+  </link>
 </robot>

Commit message: fix: Pioneer3 DX parameters

File: urdf/microbot_01_base.xacro (robot description, xacro)
@@ -26,6 +26,6 @@
   <xacro:property name="laser_w" value="0.06" />
   <xacro:property name="laser_h" value="0.06" />
-  <xacro:property name="laser_x" value="-0.0475" />
-  <xacro:property name="laser_z" value="${body_h}" />
+  <xacro:property name="laser_x" value="0.17" />
+  <xacro:property name="laser_z" value="0.1075" />
   <joint name="laser_joint" type="fixed">
     <origin xyz="${laser_x} 0 ${laser_z}" rpy="0 0 0"/>
